Commit message: made gripper interchangable

File: src/robotiq/robotiq_2f_140_gripper_visualization/urdf/robotiq_arg2f_140_model.xacro (robot description, xacro)
@@ -2,4 +2,5 @@
 <robot name="robotiq_arg2f_140_model" xmlns:xacro="http://ros.org/wiki/xacro">
   <xacro:include filename="$(find robotiq_2f_140_gripper_visualization)/urdf/robotiq_arg2f_140_model_macro.xacro" />
+  <!-- <link name="tool0"/> -->
   <xacro:robotiq_arg2f_140 prefix="" parent="tool0"/>
 </robot>

File: src/robotiq/robotiq_2f_140_gripper_visualization/urdf/robotiq_arg2f_140_model_macro.xacro (robot description, xacro)
@@ -2,4 +2,5 @@
 <robot xmlns:xacro="http://ros.org/wiki/xacro">
   <xacro:include filename="$(find robotiq_2f_140_gripper_visualization)/urdf/robotiq_arg2f_transmission.xacro" />
+  <xacro:include filename="$(find robotiq_2f_140_gripper_visualization)/urdf/robotiq_arg2f.xacro" />
   <xacro:macro name="outer_knuckle" params="prefix fingerprefix stroke">
     <link name="${prefix}${fingerprefix}_outer_knuckle">
@@ -181,5 +182,4 @@
     </joint>
   </xacro:macro>
-  <xacro:include filename="$(find robotiq_2f_140_gripper_visualization)/urdf/robotiq_arg2f.xacro" />
   <xacro:macro name="finger_joint" params="prefix">
     <joint name="${prefix}finger_joint" type="revolute">
@@ -212,11 +212,11 @@
   <xacro:macro name="robotiq_arg2f_140" params="prefix parent">
     <xacro:robotiq_arg2f_base_link prefix="${prefix}"/>
-    <xacro:finger_links prefix="${prefix}" fingerprefix="left" stroke="85"/>
-    <xacro:finger_links prefix="${prefix}" fingerprefix="right" stroke="85"/>
+    <xacro:finger_links prefix="${prefix}" fingerprefix="left" stroke="140"/>
+    <xacro:finger_links prefix="${prefix}" fingerprefix="right" stroke="140"/>
     <xacro:finger_joint prefix="${prefix}"/>
     <xacro:right_outer_knuckle_joint prefix="${prefix}"/>
     <xacro:robotiq_arg2f_transmission prefix="${prefix}"/>
-    <xacro:world_joint prefix="${prefix} ${parent}"/>
-      <origin xyz="0 0 0" rpy="0 0 0" />
+    <xacro:world_joint prefix="${prefix}" parent="${parent}">
+      <origin xyz="0 0 0" rpy="0 0 ${pi/2}" />
     </xacro:world_joint>
   </xacro:macro>

File: src/robotiq/robotiq_2f_85_gripper_visualization/urdf/robotiq_arg2f_85_model.xacro (robot description, xacro)
@@ -2,4 +2,5 @@
 <robot name="robotiq_arg2f_85_model" xmlns:xacro="http://ros.org/wiki/xacro">
   <xacro:include filename="$(find robotiq_2f_85_gripper_visualization)/urdf/robotiq_arg2f_85_model_macro.xacro" />
+  <link name="tool0"/>
   <xacro:robotiq_arg2f_85 prefix="" parent="tool0"/>
 </robot>

File: src/robotiq/robotiq_2f_85_gripper_visualization/urdf/robotiq_arg2f_85_model_macro.xacro (robot description, xacro)
@@ -5,9 +5,9 @@
   <xacro:macro name="outer_knuckle" params="prefix fingerprefix stroke">
     <link name="${prefix}${fingerprefix}_outer_knuckle">
-      <!--<inertial>
+      <inertial>
         <origin xyz="-0.000200000000003065 0.0199435877845359 0.0292245259211331" rpy="0 0 0" />
         <mass value="0.00853198276973456" />
         <inertia ixx="2.89328108496468E-06" ixy="-1.57935047237397E-19" ixz="-1.93980378593255E-19" iyy="1.86719750325683E-06" iyz="-1.21858577871576E-06" izz="1.21905238907251E-06" />
-        </inertial> -->
+      </inertial>
       <visual>
         <origin xyz="0 0 0" rpy="0 0 0" />
@@ -29,9 +29,9 @@
   <xacro:macro name="outer_finger" params="prefix fingerprefix stroke">
     <link name="${prefix}${fingerprefix}_outer_finger">
-      <!--<inertial>
+      <inertial>
         <origin xyz="0.00030115855001899 0.0373907951953854 -0.0208027427000385" rpy="0 0 0" />
         <mass value="0.022614240507152" />
         <inertia ixx="1.52518312458174E-05" ixy="9.76583423954399E-10" ixz="-5.43838577022588E-10" iyy="6.17694243867776E-06" iyz="6.78636130740228E-06" izz="1.16494917907219E-05" />
-        </inertial> -->
+      </inertial>
       <visual>
         <origin xyz="0 0 0" rpy="0 0 0" />
@@ -53,9 +53,9 @@
   <xacro:macro name="inner_knuckle" params="prefix fingerprefix stroke">
     <link name="${prefix}${fingerprefix}_inner_knuckle">
-      <!--<inertial>
+      <inertial>
         <origin xyz="0.000123011831763771 0.0507850843201817 0.00103968640075166" rpy="0 0 0" />
        <mass value="0.0271177346495152" />
         <inertia ixx="2.61910379223783E-05" ixy="-2.43616858946494E-07" ixz="-6.37789906117123E-09" iyy="2.8270243746167E-06" iyz="-5.37200748039765E-07" izz="2.83695868220296E-05" />
-        </inertial> -->
+      </inertial>
       <visual>
         <origin xyz="0 0 0" rpy="0 0 0" />
@@ -77,9 +77,9 @@
   <xacro:macro name="inner_finger" params="prefix fingerprefix stroke">
     <link name="${prefix}${fingerprefix}_inner_finger">
-      <!--<inertial>
+      <inertial>
         <origin xyz="0.000299999999999317 0.0160078233491243 -0.0136945669206257" rpy="0 0 0" />
         <mass value="0.0104003125914103" />
         <inertia ixx="2.71909453810972E-06" ixy="1.35402465472579E-21" ixz="-7.1817349065269E-22" iyy="7.69100314106116E-07" iyz="6.74715432769696E-07" izz="2.30315190420171E-06" />
-        </inertial> -->
+      </inertial>
       <visual>
         <origin xyz="0 0 0" rpy="0 0 0" />
@@ -195,5 +195,5 @@
     <xacro:right_outer_knuckle_joint prefix="${prefix}"/>
     <xacro:robotiq_arg2f_transmission prefix="${prefix}"/>
-    <xacro:world_joint prefix="${prefix} ${parent}"/>
+    <xacro:world_joint prefix="${prefix} ${parent}">
       <origin xyz="0 0 0" rpy="0 0 0" />
     </xacro:world_joint>

File: src/ur_description/urdf/ur.xacro (robot description, xacro)
@@ -6,6 +6,6 @@
    <xacro:include filename="$(find ur_description)/urdf/ur_macro.xacro"/>
    <!-- <xacro:include filename="$(find ur_description)/urdf/robotiq_2f_85.urdf.xacro"/> -->
-   <!-- <xacro:include filename="$(find robotiq_2f_85_gripper_visualization)/urdf/robotiq_arg2f_85_model.xacro"/> -->
-   <xacro:include filename="$(find robotiq_2f_140_gripper_visualization)/urdf/robotiq_arg2f_140_model.xacro"/>
+   <xacro:include filename="$(find robotiq_2f_85_gripper_visualization)/urdf/robotiq_arg2f_85_model_macro.xacro"/>
+   <xacro:include filename="$(find robotiq_2f_140_gripper_visualization)/urdf/robotiq_arg2f_140_model_macro.xacro"/>
    <xacro:include filename="$(find ur_description)/urdf/real_descr.urdf.xacro"/>
    <!-- <xacro:include filename="$(find ur_description)/urdf/zed_descr.urdf.xacro"/>  -->
@@ -13,4 +13,5 @@
    <!-- the default value should raise an error in case this was called without defining the type -->
    <xacro:arg name="ur_type" default="ur5e"/>
+   <xacro:arg name="gripper_type" default="140"/>
    <!-- parameters -->
    <xacro:arg name="tf_prefix" default="" />
@@ -96,4 +97,10 @@
      <origin xyz="0 0 0" rpy="0 0 0" />          <!-- position robot in the world -->
    </xacro:ur_robot>
+  <xacro:if value="${'$(arg gripper_type)'=='140'}">
+   <xacro:robotiq_arg2f_140 prefix="" parent="tool0"/>
+  </xacro:if>
+  <xacro:if value="${'$(arg gripper_type)'=='85'}">
+   <xacro:robotiq_arg2f_85 prefix="" parent="tool0"/>
+  </xacro:if>
   <xacro:if value="$(arg sim_gazebo)">
     <!-- Gazebo plugins -->

File: src/ur_description/urdf/ur_gripper.ros2_control.xacro (robot description, xacro)
@@ -7,6 +7,5 @@
     sim_ignition:=false
     headless_mode:=false
-    initial_positions:=${dict(shoulder_pan_joint=0.0,shoulder_lift_joint=-1.57,elbow_joint=0.0,wrist_1_joint=-1.57,wrist_2_joint=0.0,wrist_3_joint=0.0)}
-    use_tool_communication:=false
+    initial_positions
     script_filename output_recipe_filename
     input_recipe_filename tf_prefix
@@ -160,5 +159,5 @@
         <state_interface name="effort"/>
       </joint>
-      <joint name="robotiq_85_left_knuckle_joint">
+      <joint name="finger_joint">
           <command_interface name="position" />
           <state_interface name="position">
@@ -169,39 +168,29 @@
           <state_interface name="effort"/>
       </joint>
-      <joint name="robotiq_85_right_knuckle_joint">
-          <param name="mimic">robotiq_85_left_knuckle_joint</param>
-          <param name="multiplier">-1</param>
-          <command_interface name="position" />
-          <state_interface name="velocity"/>
-          <state_interface name="position"/>
-          <state_interface name="effort"/>
-      </joint>
-      <joint name="robotiq_85_left_inner_knuckle_joint">
-          <param name="mimic">robotiq_85_left_knuckle_joint</param>
-          <param name="multiplier">1</param>
-          <command_interface name="position" />
-          <state_interface name="velocity"/>
-          <state_interface name="position"/>
-          <state_interface name="effort"/>
-      </joint>
-      <joint name="robotiq_85_right_inner_knuckle_joint">
-          <param name="mimic">robotiq_85_left_knuckle_joint</param>
-          <param name="multiplier">-1</param>
-          <command_interface name="position" />
-          <state_interface name="velocity"/>
-          <state_interface name="position"/>
-          <state_interface name="effort"/>
-      </joint>
-      <joint name="robotiq_85_left_finger_tip_joint">
-          <param name="mimic">robotiq_85_left_knuckle_joint</param>
-          <param name="multiplier">-1</param>
-          <command_interface name="position" />
-          <state_interface name="velocity"/>
-          <state_interface name="position"/>
-          <state_interface name="effort"/>
-      </joint>
-      <joint name="robotiq_85_right_finger_tip_joint">
-          <param name="mimic">robotiq_85_left_knuckle_joint</param>
-          <param name="multiplier">1</param>
+      <joint name="right_outer_knuckle_joint">
+          <command_interface name="position" />
+          <state_interface name="velocity"/>
+          <state_interface name="position"/>
+          <state_interface name="effort"/>
+      </joint>
+      <joint name="left_inner_knuckle_joint">
+          <command_interface name="position" />
+          <state_interface name="velocity"/>
+          <state_interface name="position"/>
+          <state_interface name="effort"/>
+      </joint>
+      <joint name="right_inner_knuckle_joint">
+          <command_interface name="position" />
+          <state_interface name="velocity"/>
+          <state_interface name="position"/>
+          <state_interface name="effort"/>
+      </joint>
+      <joint name="left_finger_joint">
+          <command_interface name="position" />
+          <state_interface name="velocity"/>
+          <state_interface name="position"/>
+          <state_interface name="effort"/>
+      </joint>
+      <joint name="right_finger_joint">
           <command_interface name="position" />
           <state_interface name="velocity"/>

File: src/ur_description/urdf/ur_macro.xacro (robot description, xacro)
@@ -63,5 +63,5 @@
     sim_ignition:=false
     headless_mode:=false
-    initial_positions:=${dict(shoulder_pan_joint=0.0,shoulder_lift_joint=-1.57,elbow_joint=0.0,wrist_1_joint=-1.57,wrist_2_joint=0.0,wrist_3_joint=0.0)}
+    initial_positions
     use_tool_communication:=false
     tool_voltage:=0
@@ -94,7 +94,7 @@
     <xacro:if value="${generate_ros2_control_tag}">
       <!-- ros2 control include -->
-      <xacro:include filename="$(find ur_description)/urdf/ur_gripper.ros2_control.xacro" />
+      <!-- <xacro:include filename="$(find ur_description)/urdf/ur_gripper.ros2_control.xacro" /> -->
       <!-- ros2 control instance -->
-      <xacro:ur_ros2_control
+      <!-- <xacro:ur_ros2_control
         name="${name}"
         use_fake_hardware="${use_fake_hardware}"
@@ -126,5 +126,5 @@
         non_blocking_read="${non_blocking_read}"
         keep_alive_count="${keep_alive_count}"
-        />
+        /> -->
     </xacro:if>
     <!-- Add URDF transmission elements (for ros_control) -->
